Commit message: flip camera orientation and update link collision mesh

File: end_effectors/nikon_d5600_support/urdf/d5600_macro.xacro (robot description, xacro)
@@ -22,5 +22,5 @@
     <!-- Camera TCP Defined as the center point on the camera lens-->
     <joint name="${prefix}camera_link-camera_tcp" type="fixed">
-        <origin xyz="0.02222 0 0.18415" rpy="0 0 0"/>
+        <origin xyz="0.02222 0 0.18415" rpy="0 0 3.1415"/>
         <parent link="${prefix}camera_link"/>
         <child link="${prefix}camera_tcp"/>

File: end_effectors/nikon_d5600_support/urdf/gp7_d5600.xacro (robot description, xacro)
@@ -9,5 +9,5 @@
     <xacro:nikon_d5600 prefix=""/>
     <joint name="tool0-camera_link" type="fixed">
-        <origin xyz="0 0 0" rpy="0 0 0"/>
+        <origin xyz="0 0 0" rpy="0 0 3.1415"/>
         <parent link="tool0"/>
         <child link="camera_link"/>
