Commit message: Simplify Robot Cart Model

File: environment/robot_cart/urdf/cart_macro.xacro (robot description, xacro)
@@ -7,5 +7,5 @@
             <origin xyz="0 0 0" rpy="0 0 0" />
             <geometry>
-                <mesh filename="package://robot_cart/meshes/robot_cart_visual_1.stl"/>
+                <mesh filename="package://robot_cart/meshes/robot_cart_visual_back.stl"/>
             </geometry>
             <material name="table">
@@ -16,5 +16,27 @@
             <origin xyz="0 0 0" rpy="0 0 0" />
             <geometry>
-                <mesh filename="package://robot_cart/meshes/robot_cart_collision.stl"/>
+                <mesh filename="package://robot_cart/meshes/robot_cart_visual_back.stl"/>
+            </geometry>
+        </collision>
+    </link>
+    <joint name="cart_link-cart_base" type="fixed">
+        <origin xyz="0.3 0 -0.05" rpy="0 0 0"/>
+        <parent link="${prefix}cart_link"/>
+        <child link="${prefix}cart_base"/>
+    </joint>
+    <link name="${prefix}cart_base">
+        <visual>
+            <origin xyz="0 0 0" rpy="0 0 0" />
+            <geometry>
+                <box size="1.2 1.2 0.1" />
+            </geometry>
+            <material name="table">
+                <color rgba="0.8 0.8 0.8 1"/>
+            </material>
+        </visual>
+        <collision>
+            <origin xyz="0 0 0" rpy="0 0 0" />
+            <geometry>
+                <box size="1 1 0.1" />
             </geometry>
         </collision>

Commit message: Add Cart Backing Collision File

File: environment/robot_cart/urdf/cart_macro.xacro (robot description, xacro)
@@ -16,5 +16,5 @@
             <origin xyz="0 0 0" rpy="0 0 0" />
             <geometry>
-                <mesh filename="package://robot_cart/meshes/robot_cart_visual_back.stl"/>
+                <mesh filename="package://robot_cart/meshes/robot_cart_collision_back.stl"/>
             </geometry>
         </collision>
